Commit message: remove the trans file and include the transmissions within the urdf xacro Changed to Position hardware interface and JointTrajectoryController

File: src/robotic_arm_description/urdf/robotic_arm.xacro (robot description, xacro)
@@ -2,5 +2,4 @@
 <robot name="robotic_arm" xmlns:xacro="http://www.ros.org/wiki/xacro">
 <xacro:include filename="$(find robotic_arm_description)/urdf/materials.xacro" />
-<xacro:include filename="$(find robotic_arm_description)/urdf/robotic_arm.trans" />
 <xacro:include filename="$(find robotic_arm_description)/urdf/robotic_arm.gazebo" />
 <link name="world"/>
@@ -174,5 +173,7 @@
   <child link="taco_1"/>
   <axis xyz="1.0 0.0 0.0"/>
-  <limit upper="0.108" lower="-0.054" effort="100" velocity="100"/>
+  <limit upper="0.108" lower="-0.054" effort="100" velocity="1.0"/>
+  <hardwareInterface>hardware_interface/PositionJointInterface</hardwareInterface>
+  <controllerType>ros2_controllers/JointTrajectoryController</controllerType>
 </joint>
 <joint name="shoulder_link_to_taco" type="revolute">
@@ -181,5 +182,7 @@
   <child link="shoulder_link_1"/>
   <axis xyz="-1.0 -0.0 -0.0"/>
-  <limit upper="1.637119" lower="-0.261799" effort="100" velocity="100"/>
+  <limit upper="1.637119" lower="-0.261799" effort="100" velocity="1.0"/>
+  <hardwareInterface>hardware_interface/PositionJointInterface</hardwareInterface>
+  <controllerType>ros2_controllers/JointTrajectoryController</controllerType>
 </joint>
 <joint name="elbow_link_to_shoulder_link" type="revolute">
@@ -188,5 +191,7 @@
   <child link="elbow_link_1"/>
   <axis xyz="-1.0 0.0 -0.0"/>
-  <limit upper="0.959931" lower="-1.047198" effort="100" velocity="100"/>
+  <limit upper="0.959931" lower="-1.047198" effort="100" velocity="1.0"/>
+  <hardwareInterface>hardware_interface/PositionJointInterface</hardwareInterface>
+  <controllerType>ros2_controllers/JointTrajectoryController</controllerType>
 </joint>
 <joint name="bevel_housing_to_elbow_link" type="revolute">
@@ -195,5 +200,7 @@
   <child link="bevel_housing_1"/>
   <axis xyz="-1.0 0.0 -0.0"/>
-  <limit upper="1.570796" lower="-1.570796" effort="100" velocity="100"/>
+  <limit upper="1.570796" lower="-1.570796" effort="100" velocity="1.0"/>
+  <hardwareInterface>hardware_interface/PositionJointInterface</hardwareInterface>
+  <controllerType>ros2_controllers/JointTrajectoryController</controllerType>
 </joint>
 <joint name="wrist_link_to_bevel_housing" type="revolute">
@@ -202,5 +209,7 @@
   <child link="wrist_link_1"/>
   <axis xyz="0.0 -0.999855 -0.017012"/>
-  <limit upper="3.141593" lower="0.0" effort="100" velocity="100"/>
+  <limit upper="3.141593" lower="0.0" effort="100" velocity="1.0"/>
+  <hardwareInterface>hardware_interface/PositionJointInterface</hardwareInterface>
+  <controllerType>ros2_controllers/JointTrajectoryController</controllerType>
 </joint>
 <joint name="end_effector_base_to_wrist_link" type="fixed">
@@ -214,5 +223,7 @@
   <child link="moving_claw_1"/>
   <axis xyz="1.0 0.0 -0.0"/>
-  <limit upper="0.25" lower="0.0" effort="100" velocity="100"/>
+  <limit upper="0.25" lower="0.0" effort="100" velocity="1.0"/>
+  <hardwareInterface>hardware_interface/PositionJointInterface</hardwareInterface>
+  <controllerType>ros2_controllers/JointTrajectoryController</controllerType>
 </joint>
 </robot>

Commit message: change the way mesh files are linked

File: src/robotic_arm_description/urdf/robotic_arm.xacro (robot description, xacro)
@@ -17,5 +17,5 @@
     <origin xyz="0 0 0" rpy="0 0 0"/>
     <geometry>
-      <mesh filename="file://$(find robotic_arm_description)/meshes/base_link.stl" scale="0.001 0.001 0.001"/>
+      <mesh filename="package://robotic_arm_description/meshes/base_link.stl" scale="0.001 0.001 0.001"/>
     </geometry>
     <material name="grey"/>
@@ -24,5 +24,5 @@
     <origin xyz="0 0 0" rpy="0 0 0"/>
     <geometry>
-      <mesh filename="file://$(find robotic_arm_description)/meshes/base_link.stl" scale="0.001 0.001 0.001"/>
+      <mesh filename="package://robotic_arm_description/meshes/base_link.stl" scale="0.001 0.001 0.001"/>
     </geometry>
   </collision>
@@ -37,5 +37,5 @@
     <origin xyz="-0.25 -0.023 -0.0275" rpy="0 0 0"/>
     <geometry>
-      <mesh filename="file://$(find robotic_arm_description)/meshes/taco_1.stl" scale="0.001 0.001 0.001"/>
+      <mesh filename="package://robotic_arm_description/meshes/taco_1.stl" scale="0.001 0.001 0.001"/>
     </geometry>
     <material name="silver"/>
@@ -44,5 +44,5 @@
     <origin xyz="-0.25 -0.023 -0.0275" rpy="0 0 0"/>
     <geometry>
-      <mesh filename="file://$(find robotic_arm_description)/meshes/taco_1.stl" scale="0.001 0.001 0.001"/>
+      <mesh filename="package://robotic_arm_description/meshes/taco_1.stl" scale="0.001 0.001 0.001"/>
     </geometry>
   </collision>
@@ -57,5 +57,5 @@
     <origin xyz="-0.2763 -0.054 -0.13" rpy="0 0 0"/>
     <geometry>
-      <mesh filename="file://$(find robotic_arm_description)/meshes/shoulder_link_1.stl" scale="0.001 0.001 0.001"/>
+      <mesh filename="package://robotic_arm_description/meshes/shoulder_link_1.stl" scale="0.001 0.001 0.001"/>
     </geometry>
     <material name="grey"/>
@@ -64,5 +64,5 @@
     <origin xyz="-0.2763 -0.054 -0.13" rpy="0 0 0"/>
     <geometry>
-      <mesh filename="file://$(find robotic_arm_description)/meshes/shoulder_link_1.stl" scale="0.001 0.001 0.001"/>
+      <mesh filename="package://robotic_arm_description/meshes/shoulder_link_1.stl" scale="0.001 0.001 0.001"/>
     </geometry>
   </collision>
@@ -77,5 +77,5 @@
     <origin xyz="-0.2413 -0.020061 -0.635362" rpy="0 0 0"/>
     <geometry>
-      <mesh filename="file://$(find robotic_arm_description)/meshes/elbow_link_1.stl" scale="0.001 0.001 0.001"/>
+      <mesh filename="package://robotic_arm_description/meshes/elbow_link_1.stl" scale="0.001 0.001 0.001"/>
     </geometry>
     <material name="grey"/>
@@ -84,5 +84,5 @@
     <origin xyz="-0.2413 -0.020061 -0.635362" rpy="0 0 0"/>
     <geometry>
-      <mesh filename="file://$(find robotic_arm_description)/meshes/elbow_link_1.stl" scale="0.001 0.001 0.001"/>
+      <mesh filename="package://robotic_arm_description/meshes/elbow_link_1.stl" scale="0.001 0.001 0.001"/>
     </geometry>
   </collision>
@@ -97,5 +97,5 @@
     <origin xyz="-0.274 -0.564482 -0.644625" rpy="0 0 0"/>
     <geometry>
-      <mesh filename="file://$(find robotic_arm_description)/meshes/bevel_housing_1.stl" scale="0.001 0.001 0.001"/>
+      <mesh filename="package://robotic_arm_description/meshes/bevel_housing_1.stl" scale="0.001 0.001 0.001"/>
     </geometry>
     <material name="silver"/>
@@ -104,5 +104,5 @@
     <origin xyz="-0.274 -0.564482 -0.644625" rpy="0 0 0"/>
     <geometry>
-      <mesh filename="file://$(find robotic_arm_description)/meshes/bevel_housing_1.stl" scale="0.001 0.001 0.001"/>
+      <mesh filename="package://robotic_arm_description/meshes/bevel_housing_1.stl" scale="0.001 0.001 0.001"/>
     </geometry>
   </collision>
@@ -117,5 +117,5 @@
     <origin xyz="-0.2235 -0.619234 -0.645556" rpy="0 0 0"/>
     <geometry>
-      <mesh filename="file://$(find robotic_arm_description)/meshes/wrist_link_1.stl" scale="0.001 0.001 0.001"/>
+      <mesh filename="package://robotic_arm_description/meshes/wrist_link_1.stl" scale="0.001 0.001 0.001"/>
     </geometry>
     <material name="grey"/>
@@ -124,5 +124,5 @@
     <origin xyz="-0.2235 -0.619234 -0.645556" rpy="0 0 0"/>
     <geometry>
-      <mesh filename="file://$(find robotic_arm_description)/meshes/wrist_link_1.stl" scale="0.001 0.001 0.001"/>
+      <mesh filename="package://robotic_arm_description/meshes/wrist_link_1.stl" scale="0.001 0.001 0.001"/>
     </geometry>
   </collision>
@@ -137,5 +137,5 @@
     <origin xyz="-0.16875 -0.630062 -0.655742" rpy="0 0 0"/>
     <geometry>
-      <mesh filename="file://$(find robotic_arm_description)/meshes/end_effector_base_1.stl" scale="0.001 0.001 0.001"/>
+      <mesh filename="package://robotic_arm_description/meshes/end_effector_base_1.stl" scale="0.001 0.001 0.001"/>
     </geometry>
     <material name="silver"/>
@@ -144,5 +144,5 @@
     <origin xyz="-0.16875 -0.630062 -0.655742" rpy="0 0 0"/>
     <geometry>
-      <mesh filename="file://$(find robotic_arm_description)/meshes/end_effector_base_1.stl" scale="0.001 0.001 0.001"/>
+      <mesh filename="package://robotic_arm_description/meshes/end_effector_base_1.stl" scale="0.001 0.001 0.001"/>
     </geometry>
   </collision>
@@ -157,5 +157,5 @@
     <origin xyz="-0.15025 -0.641231 -0.645931" rpy="0 0 0"/>
     <geometry>
-      <mesh filename="file://$(find robotic_arm_description)/meshes/moving_claw_1.stl" scale="0.001 0.001 0.001"/>
+      <mesh filename="package://robotic_arm_description/meshes/moving_claw_1.stl" scale="0.001 0.001 0.001"/>
     </geometry>
     <material name="grey"/>
@@ -164,5 +164,5 @@
     <origin xyz="-0.15025 -0.641231 -0.645931" rpy="0 0 0"/>
     <geometry>
-      <mesh filename="file://$(find robotic_arm_description)/meshes/moving_claw_1.stl" scale="0.001 0.001 0.001"/>
+      <mesh filename="package://robotic_arm_description/meshes/moving_claw_1.stl" scale="0.001 0.001 0.001"/>
     </geometry>
   </collision>
