Commit message: THINGS I DID TO MAKE IT WORK

File: src/my_robot_canopen_control/urdf/robotic_arm.ros2_control.xacro (robot description, xacro)
@@ -6,5 +6,7 @@
       master_config
       can_interface_name
-      master_bin">
+      master_bin
+      initial_positions_file">
+        <xacro:property name="initial_positions" value="${xacro.load_yaml(initial_positions_file)['initial_positions']}"/>
         <ros2_control name="${name}" type="system">
             <hardware>
@@ -17,17 +19,40 @@
             <joint name="shoulder_link_to_taco">
                 <param name="device_name">shoulder_link_to_taco</param>
-                <state_interface name="position" />
+                <command_interface name="position"/>
+                <state_interface name="position">
+                  <param name="initial_value">${initial_positions['shoulder_link_to_taco']}</param>
+                </state_interface>
+                <state_interface name="velocity">
+                  <param name="initial_value">0.0</param>
+                </state_interface>
             </joint>
             <joint name="elbow_link_to_shoulder_link">
                 <param name="device_name">elbow_link_to_shoulder_link</param>
-                <state_interface name="position" />
+                <command_interface name="position"/>
+                <state_interface name="position">
+                  <param name="initial_value">${initial_positions['elbow_link_to_shoulder_link']}</param>
+                </state_interface>
+                <state_interface name="velocity">
+                  <param name="initial_value">0.0</param>
+                </state_interface>
             </joint>
             <joint name="bevel_housing_to_elbow_link">
                 <param name="device_name">bevel_housing_to_elbow_link</param>
-                <state_interface name="position" />
+                <command_interface name="position"/>
+                <state_interface name="position">
+                  <param name="initial_value">${initial_positions['bevel_housing_to_elbow_link']}</param>
+                </state_interface>
+                <state_interface name="velocity">
+                  <param name="initial_value">0.0</param>
+                </state_interface>
             </joint>
             <joint name="wrist_link_to_bevel_housing">
                 <param name="device_name">wrist_link_to_bevel_housing</param>
-                <state_interface name="position" />
+                <state_interface name="position">
+                  <param name="initial_value">${initial_positions['wrist_link_to_bevel_housing']}</param>
+                </state_interface>
+                <state_interface name="velocity">
+                  <param name="initial_value">0.0</param>
+                </state_interface>
             </joint>
         </ros2_control>

File: src/my_robot_canopen_control/urdf/robotic_arm.urdf.xacro (robot description, xacro)
@@ -1,4 +1,5 @@
 <?xml version="1.0"?>
 <robot xmlns:xacro="http://wiki.ros.org/xacro" name="robotic_arm_v1">
+    <xacro:arg name="initial_positions_file" default="initial_positions.yaml" />
     <xacro:include filename="$(find my_robot_description)/urdf/robotic_arm.xacro"/>
     <xacro:include filename="$(find my_robot_canopen_control)/urdf/robotic_arm.ros2_control.xacro"/>
@@ -8,4 +9,5 @@
         master_config="$(find my_robot_canopen_control)/config/robot_control/master.dcf"
         can_interface_name="can0"
-        master_bin="" />
+        master_bin=""
+        initial_positions_file="$(arg initial_positions_file)"/>
 </robot>

File: src/my_robot_description/urdf/robotic_arm.xacro (robot description, xacro)
@@ -48,5 +48,5 @@
     </collision>
   </link>
-  <joint name="taco_to_base_link" type="prismatic">
+  <joint name="taco_to_base_link" type="fixed">
     <origin xyz="0.25 0.023 0.0275" rpy="0 0 0"/>
     <parent link="base_link"/>
@@ -213,5 +213,5 @@
     </collision>
   </link>
-  <joint name="moving_claw_to_end_effector_base" type="prismatic">
+  <joint name="moving_claw_to_end_effector_base" type="fixed">
     <origin xyz="-0.0185 0.011169 -0.009811" rpy="0 0 0"/>
     <parent link="end_effector_base_1"/>

File: src/my_robot_moveit_config/config/robotic_arm.urdf.xacro (robot description, xacro)
@@ -1,9 +1,13 @@
 <?xml version="1.0"?>
-<robot xmlns:xacro="http://www.ros.org/wiki/xacro" name="robotic_arm">
+<robot xmlns:xacro="http://wiki.ros.org/xacro" name="robotic_arm_v1">
     <xacro:arg name="initial_positions_file" default="initial_positions.yaml" />
-    <!-- Import robotic_arm urdf file -->
-    <xacro:include filename="$(find my_robot_description)/urdf/robotic_arm.xacro" />
-    <!-- Import control_xacro -->
-    <xacro:include filename="robotic_arm.ros2_control.xacro" />
-    <xacro:robotic_arm_ros2_control name="FakeSystem" initial_positions_file="$(arg initial_positions_file)"/>
+    <xacro:include filename="$(find my_robot_description)/urdf/robotic_arm.xacro"/>
+    <xacro:include filename="$(find my_robot_canopen_control)/urdf/robotic_arm.ros2_control.xacro"/>
+    <xacro:robot_control_control
+        name="robotic_arm_v1"
+        bus_config="$(find my_robot_canopen_control)/config/robot_control/bus.yml"
+        master_config="$(find my_robot_canopen_control)/config/robot_control/master.dcf"
+        can_interface_name="can0"
+        master_bin=""
+        initial_positions_file="$(arg initial_positions_file)"/>
 </robot>
