Commit message: fix axis alignment of wrist_link_to_bevel_housing join in the URDF

File: src/my_robot_description/urdf/robotic_arm.xacro (robot description, xacro)
@@ -164,5 +164,5 @@
     <parent link="bevel_housing_1"/>
     <child link="wrist_link_1"/>
-    <axis xyz="0.0 -0.999855 -0.017012"/>
+    <axis xyz="0.0 -0.1 0.0"/>
     <limit upper="3.141593" lower="0.0" effort="100" velocity="1.0"/>
     <hardwareInterface>hardware_interface/PositionJointInterface</hardwareInterface>

Commit message: control via keyboard working

File: src/my_robot_description/urdf/robotic_arm.xacro (robot description, xacro)
@@ -81,5 +81,5 @@
     <child link="shoulder_link_1"/>
     <axis xyz="-1.0 -0.0 -0.0"/>
-    <limit upper="1.637119" lower="-0.261799" effort="100" velocity="1.0"/>
+    <limit upper="3.14" lower="-3.14" effort="100" velocity="1.0"/>
     <hardwareInterface>hardware_interface/PositionJointInterface</hardwareInterface>
   </joint>
@@ -109,5 +109,5 @@
     <child link="elbow_link_1"/>
     <axis xyz="-1.0 0.0 -0.0"/>
-    <limit upper="0.959931" lower="-1.047198" effort="100" velocity="1.0"/>
+    <limit upper="3.14" lower="-3.14" effort="100" velocity="1.0"/>
     <hardwareInterface>hardware_interface/PositionJointInterface</hardwareInterface>
   </joint>
@@ -137,5 +137,5 @@
     <child link="bevel_housing_1"/>
     <axis xyz="-1.0 0.0 -0.0"/>
-    <limit upper="1.570796" lower="-1.570796" effort="100" velocity="1.0"/>
+    <limit upper="3.14" lower="-3.14" effort="100" velocity="1.0"/>
     <hardwareInterface>hardware_interface/PositionJointInterface</hardwareInterface>
   </joint>
@@ -165,5 +165,5 @@
     <child link="wrist_link_1"/>
     <axis xyz="0.0 -0.1 0.0"/>
-    <limit upper="3.141593" lower="0.0" effort="100" velocity="1.0"/>
+    <limit upper="3.141593" lower="-3.14" effort="100" velocity="1.0"/>
     <hardwareInterface>hardware_interface/PositionJointInterface</hardwareInterface>
   </joint>

Commit message: update joint limits

File: src/my_robot_description/urdf/robotic_arm.xacro (robot description, xacro)
@@ -109,5 +109,5 @@
     <child link="elbow_link_1"/>
     <axis xyz="-1.0 0.0 -0.0"/>
-    <limit upper="3.14" lower="-3.14" effort="100" velocity="1.0"/>
+    <limit upper="3.14" lower="-1.57" effort="100" velocity="1.0"/>
     <hardwareInterface>hardware_interface/PositionJointInterface</hardwareInterface>
   </joint>
